Commit message: Add full humanoid body to URDF

File: ros2_ws/src/bipedal_robot_description/urdf/bipedal.urdf (robot description, URDF)
Before this commit: robot bipedal_robot, 7 links, 6 joints
Links:
- added link head, mass 3.0; collision sphere radius=0.12; visual sphere radius=0.12
- added link left_hand, mass 0.3; collision box size=0.08 0.1 0.04; visual box size=0.08 0.1 0.04
- added link left_lower_arm, mass 0.7; collision cylinder length=0.25 radius=0.035; visual cylinder length=0.25 radius=0.035
- added link left_upper_arm, mass 1.0; collision cylinder length=0.3 radius=0.04; visual cylinder length=0.3 radius=0.04
- added link right_hand, mass 0.3; collision box size=0.08 0.1 0.04; visual box size=0.08 0.1 0.04
- added link right_lower_arm, mass 0.7; collision cylinder length=0.25 radius=0.035; visual cylinder length=0.25 radius=0.035
- added link right_upper_arm, mass 1.0; collision cylinder length=0.3 radius=0.04; visual cylinder length=0.3 radius=0.04
- link base_link: mass 10.0 -> 15.0; geometry collision box size=0.35 0.25 0.5; visual box size=0.35 0.25 0.5
- link left_foot: mass 0.5 -> 0.8; geometry collision box size=0.2 0.1 0.05; visual box size=0.2 0.1 0.05
- link left_shin: mass 1.5 -> 2.0; geometry collision cylinder length=0.35 radius=0.05; visual cylinder length=0.35 radius=0.05
- link left_thigh: mass 2.0 -> 3.0; geometry collision cylinder length=0.4 radius=0.06; visual cylinder length=0.4 radius=0.06
- link right_foot: mass 0.5 -> 0.8; geometry collision box size=0.2 0.1 0.05; visual box size=0.2 0.1 0.05
- link right_shin: mass 1.5 -> 2.0; geometry collision cylinder length=0.35 radius=0.05; visual cylinder length=0.35 radius=0.05
- link right_thigh: mass 2.0 -> 3.0; geometry collision cylinder length=0.4 radius=0.06; visual cylinder length=0.4 radius=0.06
Joints:
- added joint left_elbow_joint: type fixed, parent left_upper_arm, child left_lower_arm, origin xyz=0 0 -0.3 rpy=0 0 0
- added joint left_hand_joint: type fixed, parent left_lower_arm, child left_hand, origin xyz=0 0 -0.25 rpy=0 0 0
- added joint left_shoulder_joint: type fixed, parent base_link, child left_upper_arm, origin xyz=0 0.2 0.15 rpy=0 0 0
- added joint neck_joint: type fixed, parent base_link, child head, origin xyz=0 0 0.35 rpy=0 0 0
- added joint right_elbow_joint: type fixed, parent right_upper_arm, child right_lower_arm, origin xyz=0 0 -0.3 rpy=0 0 0
- added joint right_hand_joint: type fixed, parent right_lower_arm, child right_hand, origin xyz=0 0 -0.25 rpy=0 0 0
- added joint right_shoulder_joint: type fixed, parent base_link, child right_upper_arm, origin xyz=0 -0.2 0.15 rpy=0 0 0
- joint left_hip_joint: origin xyz=-0.05 0.1 -0.3 rpy=0 0 0 -> xyz=0 0.1 -0.25 rpy=0 0 0
- joint right_hip_joint: origin xyz=-0.05 -0.1 -0.3 rpy=0 0 0 -> xyz=0 -0.1 -0.25 rpy=0 0 0
